File: PCB/GPS traacker.kicad_pcb (KiCad board)
At the start: 2 copper layers, 55 x 42 mm, 33 parts, among them J1 USB_C_Receptacle, J2 Conn_01x02_Pin, J3 Conn_Coaxial, J4 Micro_SD_Card, SW1 SW_Push, U1 TP4056-42-ESOP8, U2 AP2112K-3.3, U3 MOUDLE-SEEEDUINO-XIAO, U4 MAX-M10S

Commit message: Development files
Routing:
- net Net-(U3-PA10_A2_D2): track 29.0 -> 32.4 mm
- net Net-(U3-PA11_A3_D3): track 12.0 -> 12.8 mm
- net Net-(U3-PA4_A1_D1): track 6.42 -> 7.15 mm
Changed lines of the file:
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@@
 			(at 1 4 0)
 			(layer "F.Fab")
+			(hide yes)
 			(effects
 				(font
@@
 			(at 0 3.2 0)
 			(layer "F.Fab")
+			(hide yes)
 			(effects
 				(font
@@
 		(tags "capacitor")
 		(property "Reference" "C5"
-			(at 0 -1.43 90)
+			(at 0 1.5 90)
 			(layer "F.SilkS")
 			(effects
@@
 	)
 	(segment
-		(start 113 62.262648)
-		(end 113 60.403982)
+		(start 111.5 61.75)
+		(end 111.5 60.77587)
 		(width 0.2)
 		(layer "F.Cu")
@@
 	)
 	(segment
-		(start 122.555346 67.00753)
-		(end 117.744882 67.00753)
+		(start 124.5 65.75)
+		(end 123 67.25)
 		(width 0.2)
 		(layer "F.Cu")
@@
 	)
 	(segment
-		(start 114.237345 59.166637)
-		(end 115.333363 59.166637)
+		(start 124.5 58.06853)
+		(end 124.5 65.75)
 		(width 0.2)
 		(layer "F.Cu")
@@
 	)
 	(segment
-		(start 124.15 57.71853)
-		(end 124.15 65.412876)
+		(start 123 67.25)
+		(end 117 67.25)
 		(width 0.2)
 		(layer "F.Cu")
@@
 	)
 	(segment
-		(start 113 60.403982)
-		(end 114.237345 59.166637)
+		(start 117 67.25)
+		(end 111.5 61.75)
 		(width 0.2)
 		(layer "F.Cu")
@@
 	)
 	(segment
-		(start 122.129 55.69753)
-		(end 124.15 57.71853)
+		(start 113.109233 59.166637)
+		(end 115.333363 59.166637)
 		(width 0.2)
 		(layer "F.Cu")
@@
 	)
 	(segment
-		(start 117.744882 67.00753)
-		(end 113 62.262648)
+		(start 111.5 60.77587)
+		(end 113.109233 59.166637)
 		(width 0.2)
 		(layer "F.Cu")
@@
 	)
 	(segment
-		(start 124.15 65.412876)
-		(end 122.555346 67.00753)
+		(start 122.129 55.69753)
+		(end 124.5 58.06853)
 		(width 0.2)
 		(layer "F.Cu")
@@
 	)
 	(segment
+		(start 124.1 63.4)
+		(end 124.1 59.404265)
+		(width 0.2)
+		(layer "F.Cu")
+		(net "Net-(U3-PA11_A3_D3)")
+	)
+	(segment
 		(start 118.325 64.25)
 		(end 118.575 64.5)
@@
 	)
 	(segment
-		(start 123.75 63.75)
-		(end 123.75 59.85853)
+		(start 122.933265 58.23753)
+		(end 122.129 58.23753)
 		(width 0.2)
 		(layer "F.Cu")
@@
 	(segment
 		(start 123 64.5)
-		(end 123.75 63.75)
+		(end 124.1 63.4)
 		(width 0.2)
 		(layer "F.Cu")
@@
 	)
 	(segment
-		(start 123.75 59.85853)
-		(end 122.129 58.23753)
+		(start 124.1 59.404265)
+		(end 122.933265 58.23753)
 		(width 0.2)
 		(layer "F.Cu")
@@
 	)
 	(segment
-		(start 118.575 57.5)
-		(end 118.575 55.675184)
+		(start 118.575 54.425)
+		(end 119.84247 53.15753)
 		(width 0.2)
 		(layer "F.Cu")
@@
 	)
 	(segment
-		(start 121.092654 53.15753)
+		(start 119.84247 53.15753)
 		(end 122.129 53.15753)
 		(width 0.2)
@@
 	)
 	(segment
-		(start 118.575 55.675184)
-		(end 121.092654 53.15753)
+		(start 118.575 57.5)
+		(end 118.575 54.425)
 		(width 0.2)
 		(layer "F.Cu")
